File: PCB/main/outputs.kicad_sch (KiCad schematic)
At the start: 0 parts

Commit message: Finished initial design
Other:
- company: (none) -> University of Cape Town
Changed lines of the file:
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@@
 (kicad_sch (version 20211123) (generator eeschema)
   (paper "A4")
+  (title_block
+    (company "University of Cape Town")
+    (comment 2 "@Project EEE3088F-Team-9")
+  )
   (text "Not sure if you want this here:\n\nGP LEDS\nPushButton or 2 for testing\nUSB Connector\nTesting Connector\nJumpers for debugging and inserting signals"
     (at 126.365 86.36 0)
