File: PCB/main/main.kicad_sch (KiCad schematic)
At the start: 4 parts, among them J1 Conn_01x33_Female, J2 Conn_01x33_Female, J3 Conn_01x33_Female, J4 Conn_01x33_Female

Commit message: Finished initial design
Connections:
- net PB10 renamed BARO_SCL
- net PB11 renamed BARO_SDA
- net PC5 renamed TEMP_OUT
Changed lines of the file:
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@@
     (rev "V0.2")
     (company "University of Cape Town")
+    (comment 2 "@Project EEE3088F-Team-9")
     (comment 3 "@Checked By: ")
     (comment 4 "@Authors: David Young, Cameron Wilson, Caide Spriestersbach")
@@
     (stroke (width 0) (type default) (color 0 0 0 0))
   )
+  (wire (pts (xy 71.12 110.49) (xy 74.93 110.49))
+    (stroke (width 0) (type default) (color 0 0 0 0))
+  )
+  (wire (pts (xy 71.12 102.87) (xy 74.93 102.87))
+    (stroke (width 0) (type default) (color 0 0 0 0))
+  )
   (polyline (pts (xy 284.48 109.855) (xy 201.295 109.855))
     (stroke (width 0) (type default) (color 0 0 0 0))
@@
     (stroke (width 0) (type default) (color 0 0 0 0))
   )
+  (wire (pts (xy 71.12 113.03) (xy 74.93 113.03))
+    (stroke (width 0) (type default) (color 0 0 0 0))
+  )
   (polyline (pts (xy 201.295 109.855) (xy 201.295 165.735))
     (stroke (width 0) (type default) (color 0 0 0 0))
@@
     (stroke (width 0) (type default) (color 0 0 0 0))
   )
+  (wire (pts (xy 71.12 105.41) (xy 74.93 105.41))
+    (stroke (width 0) (type default) (color 0 0 0 0))
+  )
   (wire (pts (xy 248.285 34.29) (xy 253.365 34.29))
     (stroke (width 0) (type default) (color 0 0 0 0))
@@
   )
   (wire (pts (xy 211.455 24.13) (xy 213.995 24.13))
+    (stroke (width 0) (type default) (color 0 0 0 0))
+  )
+  (wire (pts (xy 71.12 115.57) (xy 74.93 115.57))
     (stroke (width 0) (type default) (color 0 0 0 0))
   )
@@
     (effects (font (size 1.27 1.27)) (justify left bottom))
   )
+  (label "PB11" (at 74.93 113.03 0)
+    (effects (font (size 1.27 1.27)) (justify left bottom))
+  )
   (label "PA5" (at 229.235 77.47 0)
     (effects (font (size 1.27 1.27)) (justify left bottom))
@@
     (effects (font (size 1.27 1.27)) (justify left bottom))
   )
+  (label "PC5" (at 74.93 115.57 0)
+    (effects (font (size 1.27 1.27)) (justify left bottom))
+  )
   (label "PB10" (at 211.455 97.79 0)
     (effects (font (size 1.27 1.27)) (justify left bottom))
@@
   )
   (label "PC5" (at 211.455 87.63 0)
+    (effects (font (size 1.27 1.27)) (justify left bottom))
+  )
+  (label "PB10" (at 74.93 110.49 0)
     (effects (font (size 1.27 1.27)) (justify left bottom))
   )
@@
     )
   )
+  (global_label "V3.3" (shape input) (at 74.93 105.41 0) (fields_autoplaced)
+    (effects (font (size 1.27 1.27)) (justify left))
+    (property "Intersheet References" "${INTERSHEET_REFS}" (id 0) (at 81.4555 105.3306 0)
+      (effects (font (size 1.27 1.27)) (justify left) hide)
+    )
+  )
   (global_label "1V7" (shape input) (at 137.16 50.8 0) (fields_autoplaced)
     (effects (font (size 1.27 1.27)) (justify left))
@@
     )
   )
+  (global_label "TEMP_VCC" (shape input) (at 71.12 102.87 180) (fields_autoplaced)
+    (effects (font (size 1.27 1.27)) (justify right))
+    (property "Intersheet References" "${INTERSHEET_REFS}" (id 0) (at 59.2726 102.9494 0)
+      (effects (font (size 1.27 1.27)) (justify right) hide)
+    )
+  )
+  (global_label "TEMP_OUT" (shape input) (at 71.12 115.57 180) (fields_autoplaced)
+    (effects (font (size 1.27 1.27)) (justify right))
+    (property "Intersheet References" "${INTERSHEET_REFS}" (id 0) (at 59.2726 115.4906 0)
+      (effects (font (size 1.27 1.27)) (justify right) hide)
+    )
+  )
   (global_label "MEM_VCC" (shape input) (at 133.35 50.8 180) (fields_autoplaced)
     (effects (font (size 1.27 1.27)) (justify right))
     (property "Intersheet References" "${INTERSHEET_REFS}" (id 0) (at 122.2888 50.7206 0)
+      (effects (font (size 1.27 1.27)) (justify right) hide)
+    )
+  )
+  (global_label "V3.3" (shape input) (at 74.93 102.87 0) (fields_autoplaced)
+    (effects (font (size 1.27 1.27)) (justify left))
+    (property "Intersheet References" "${INTERSHEET_REFS}" (id 0) (at 81.4555 102.7906 0)
+      (effects (font (size 1.27 1.27)) (justify left) hide)
+    )
+  )
+  (global_label "BARO_SDA" (shape input) (at 71.12 113.03 180) (fields_autoplaced)
+    (effects (font (size 1.27 1.27)) (justify right))
+    (property "Intersheet References" "${INTERSHEET_REFS}" (id 0) (at 59.2121 112.9506 0)
+      (effects (font (size 1.27 1.27)) (justify right) hide)
+    )
+  )
+  (global_label "BARO_VDD" (shape input) (at 71.12 105.41 180) (fields_autoplaced)
+    (effects (font (size 1.27 1.27)) (justify right))
+    (property "Intersheet References" "${INTERSHEET_REFS}" (id 0) (at 59.1517 105.4894 0)
+      (effects (font (size 1.27 1.27)) (justify right) hide)
+    )
+  )
+  (global_label "BARO_SCL" (shape input) (at 71.12 110.49 180) (fields_autoplaced)
+    (effects (font (size 1.27 1.27)) (justify right))
+    (property "Intersheet References" "${INTERSHEET_REFS}" (id 0) (at 59.2726 110.4106 0)
       (effects (font (size 1.27 1.27)) (justify right) hide)
     )
@@
       (reference "#PWR0112") (unit 1) (value "GND") (footprint "")
     )
+    (path "/cf6c12a4-3d95-473d-bafe-8be3892a84e9/716e8bf5-fb1a-4f84-be63-2eb75a2e1cf2"
+      (reference "#PWR?") (unit 1) (value "GND") (footprint "")
+    )
     (path "/d15c8919-7ccc-44b2-8fc4-b04c1b47b6fa/737e9f67-33d5-420a-8f8f-42955190a9f6"
       (reference "C1") (unit 1) (value "10u") (footprint "")
@@
     )
     (path "/cf6c12a4-3d95-473d-bafe-8be3892a84e9/7228bdfc-95f0-4c15-b9fb-cf288b667432"
-      (reference "U4") (unit 1) (value "TO-92_Temperature_Sensor") (footprint "")
+      (reference "U4") (unit 1) (value "LM61BIZ/NOPD_TempSensor(TO-92)") (footprint "")
     )
     (path "/cf6c12a4-3d95-473d-bafe-8be3892a84e9/8dd5d845-7e1c-4663-a6ba-2af71acfbef6"
-      (reference "U5") (unit 1) (value "C94049_Barometer") (footprint "")
+      (reference "U5") (unit 1) (value "LPS22HBTR_Barometer") (footprint "")
     )
     (path "/59b42903-2dc7-4011-ab5b-d7b81bd233c3/1f77e19d-e9a2-47dc-9090-a7adfe4813b9"

Commit message: Fiddled a bit with labels
Connections:
- net BARO_SCL renamed PB10
- net BARO_SDA renamed PB11
- net MEM_SCL renamed PB6
- net MEM_SDA renamed PB7
- net RXD_IN renamed PA9
- net TEMP_OUT renamed PC5
- net TXD_OUT renamed PA10
- no-connect marks 0 -> 1
Other:
- sheet Power ports: added 1V7, 5V, GND, USB_5V, V3.3; removed none
- sheet Sensing ports: added BARO_SCL, BARO_SDA, BARO_VDD, GND, TEMP_OUT, TEMP_VCC; removed none
- sheet microcontroller_interfacing ports: added FTDI_RST, FTDI_VDD, GND, MEM_SCL, MEM_SDA, MEM_VCC, RXD_IN, TXD_OUT; removed none
