File: PCB/main/main.kicad_sch (KiCad schematic)
At the start: 4 parts, among them J1 Conn_01x33_Female, J2 Conn_01x33_Female, J3 Conn_01x33_Female, J4 Conn_01x33_Female

Commit message: Updated all footprints of components
Connections:
- no-connect marks 1 -> 0
Other:
- sheet microcontroller_interfacing ports: added none; removed FTDI_RST

Commit message: Connected voltage supply from USB to power subsystem
Other:
- sheet microcontroller_interfacing ports: added 5V from USB; removed none
Changed lines of the file:
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@@
+    (stroke (width 0) (type default) (color 0 0 0 0))
+  )
+  (wire (pts (xy 109.855 48.895) (xy 114.3 48.895))
     (stroke (width 0) (type default) (color 0 0 0 0))
   )
@@
   (label "PF5" (at 229.235 72.39 0)
     (effects (font (size 1.27 1.27)) (justify left bottom))
+  )
+  (label "USB_5V" (at 109.855 48.895 180)
+    (effects (font (size 1.27 1.27)) (justify right bottom))
   )
   (label "USB_5V" (at 45.72 49.53 180)
@@
       (effects (font (size 1.27 1.27)) (justify right))
     )
-  )
+    (pin "5V from USB" input (at 114.3 48.895 180)
+      (effects (font (size 1.27 1.27)) (justify left))
+    )
+  )
